File: Retro6502-Mainboard.kicad_sch (KiCad schematic)
At the start: 4 parts, among them U1 W65C02SxP, U2 IS62WV2568BLL-55HLI, U3 ATF1502ASV-xAx44

Commit message: Updates
Parts:
- added U4: 27C512, Package_DIP:DIP-28_W15.24mm, symbol Memory_EPROM:27C512
- added Y2: 16MHz, Oscillator:Oscillator_SMD_SeikoEpson_SG8002CA-4Pin_7.0x5.0mm, symbol Oscillator:SG-7050CAN
Connections:
- net A0: now also U4.10 (A0)
- net A1: now also U4.9 (A1)
- net A10: now also U4.21 (A10)
- net A11: now also U4.23 (A11)
- net A12: now also U4.2 (A12)
- net A13: now also U4.26 (A13)
- net A14: now also U4.27 (A14)
- net A15: now also U4.1 (A15)
- net A2: now also U4.8 (A2)
- net A3: now also U4.7 (A3)
- net A4: now also U4.6 (A4)
- net A5: now also U4.5 (A5)
- net A6: now also U4.4 (A6)
- net A7: now also U4.3 (A7)
- net A8: now also U4.25 (A8)
- net A9: now also U4.24 (A9)
- net D0: now also U4.11 (D0)
- net D1: now also U4.12 (D1)
- net D2: now also U4.13 (D2)
- net D3: now also U4.15 (D3)
- net D4: now also U4.16 (D4)
- net D5: now also U4.17 (D5)
- net D6: now also U4.18 (D6)
- net D7: now also U4.19 (D7)
- net GND: now also U2.32 (~{OE}), U4.14 (GND), U4.22 (~{OE}), Y2.2 (GND)
- net ~{CSROM}: now also U4.20 (~{CE})
- net 1MHz: now reaches U1.35 (ϕ2)
- net 1MHz: now also U3.42 (I/O)
- net 16MHz: now reaches U3.8 (I/O)
- net 16MHz: now also Y2.3 (OUT)
- no-connect marks 0 -> 1
